Commit message: Support for Gazebo Harmonic

File: robots/summit_xl_std.urdf.xacro (robot description, xacro)
@@ -5,8 +5,8 @@
   <!-- ***************** -->
   <!-- Import RB1 base elements (base + wheels) -->
-  <xacro:include filename="$(find summit_xl_description)/urdf/bases/summit_xl_base.urdf.xacro"/>
-  <xacro:include filename="$(find summit_xl_description)/urdf/wheels/rubber_wheel.urdf.xacro"/>
-  <xacro:include filename="$(find summit_xl_description)/urdf/wheels/omni_wheel.urdf.xacro"/>
-  <xacro:include filename="$(find summit_xl_description)/urdf/structures/structure_gps.urdf.xacro"/>
+  <xacro:include filename="$(find robot_description)/urdf/bases/summit_xl_base.urdf.xacro"/>
+  <xacro:include filename="$(find robot_description)/urdf/wheels/rubber_wheel/rubber_wheel.urdf.xacro"/>
+  <xacro:include filename="$(find robot_description)/urdf/wheels/omni_wheel/omni_wheel.urdf.xacro"/>
+  <xacro:include filename="$(find robot_description)/urdf/structures/sensor_support/structure_gps.urdf.xacro"/>
   <!-- Import all available sensors -->
   <xacro:include filename="$(find robotnik_sensors)/urdf/all_sensors.urdf.xacro"/>
@@ -17,13 +17,14 @@
   <!-- Wheel parameters -->
   <!-- x,y,z in translation from base_link to the center of the wheel -->
-  <xacro:property name="wheel_offset_x" value="0.218"/>
-  <xacro:property name="wheel_offset_y" value="0.228"/>
+  <xacro:property name="wheel_offset_x" value="0.229"/>
+  <xacro:property name="wheel_offset_y" value="0.235"/>
   <xacro:property name="wheel_offset_z" value="0.0"/>
   <!-- Flag to select the high or low quality model -->
   <xacro:property name="hq" value="true"/>
-  <xacro:arg name="robot_id" default="robot"/>
+  <xacro:arg name="robot_id" default="summit_xl"/>
   <xacro:arg name="prefix" default=""/>
   <xacro:arg name="robot_ns" default=""/>
   <xacro:arg name="omni_wheels" default="false"/>
+  <xacro:arg name="use_sim_time" default="true"/>
   <!-- *************** -->
   <!-- Robots Elements -->
@@ -62,5 +63,5 @@
   </xacro:if>
   <!-- SENSORS -->
-  <xacro:sensor_robosense_helios node_namespace="$(arg robot_ns)" frame_prefix="$(arg prefix)front_laser_" parent="$(arg prefix)base_link" simulation="true" gpu="false">
+  <xacro:sensor_robosense_helios node_namespace="$(arg robot_ns)" frame_prefix="$(arg prefix)front_laser_" parent="$(arg prefix)base_link" simulation="true" gpu="true">
       <origin xyz="-0.11808 0.0 0.38509" rpy="0 0 0"/>
   </xacro:sensor_robosense_helios>
@@ -74,9 +75,9 @@
     <origin xyz="-0.24 0.095 0.625" rpy="0 0 0"/>
   </xacro:sensor_gps>
-  <xacro:sensor_imu ns="$(arg robot_ns)" prefix="$(arg prefix)imu_" parent="$(arg prefix)base_link">
+  <xacro:sensor_imu ns="$(arg robot_ns)" prefix="$(arg prefix)imu" parent="$(arg prefix)base_link">
     <origin xyz="0.0 0.0 0.0" rpy="0 0 0"/>
   </xacro:sensor_imu>
   <!-- Gazebo ros control plugins -->
-  <xacro:arg name="config_controllers" default="$(find summit_simulator)/config/summit_xl_base.yaml"/>
+  <xacro:arg name="config_controllers" default="$(find robot_description)/config/summit_controllers.yaml"/>
   <xacro:arg name="update_rate" default="100"/>
   <xacro:include filename="$(find summit_simulator)/urdf/ros2_control.urdf.xacro"/>

File: urdf/ros2_control.urdf.xacro (robot description, xacro)
@@ -3,5 +3,5 @@
   <xacro:macro name="ros2_control">
       <gazebo>
-        <plugin name="ros_control" filename="libgazebo_ros2_control.so">
+        <plugin filename="libgz_ros2_control-system.so" name="gz_ros2_control::GazeboSimROS2ControlPlugin">
           <parameters>$(arg config_controllers)</parameters>
         </plugin>
@@ -9,5 +9,5 @@
       <ros2_control name="robotnik_base_hw" type="system">
         <hardware>
-          <plugin>gazebo_ros2_control/GazeboSystem</plugin>
+           <plugin>gz_ros2_control/GazeboSimSystem</plugin>
         </hardware>
         <joint name="front_left_wheel_joint">
